File: tcg_counter/tcg_counter.kicad_sch (KiCad schematic)
At the start: 21 parts, among them J1 U.FL, P1 TC2050-IDC-430, U1 TCAL9539RTW, U3 RF430FRL152

Commit message: Added decoupling capacitors on TCAL9539RTW
Parts:
- added C11: 1uF, symbol Device:C
- added C12: 0.1uF, symbol Device:C
Connections:
- net GND: now also C11.2, C12.2
- net at C2.1, R4.1, R5.1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: now also C11.1, C12.1

Commit message: Assigned footprints
Parts:
- C11, C12: footprint (none) -> Capacitor_SMD:C_0402_1005Metric
- P1: footprint (none) -> Connector:Tag-Connect_TC2050-IDC-NL_2x05_P1.27mm_Vertical_with_bottom_clip
- R1, R4, R5: footprint (none) -> Resistor_SMD:R_0402_1005Metric
- U2: footprint (none) -> Library:D0430G02V01
Connections:
- net VDDSW: now reaches C11.1, C12.1, C2.1, R4.1, R5.1, U1.21 (VCC), U3.3 (VDDSW)
Changed lines of the file:
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@@
 	)
 	(junction
+		(at 74.93 22.86)
+		(diameter 0)
+		(color 0 0 0 0)
+	)
+	(junction
 		(at 91.44 22.86)
 		(diameter 0)
@@
 	(wire
 		(pts
+			(xy 69.85 22.86) (xy 74.93 22.86)
+		)
+		(stroke
+			(width 0)
+			(type default)
+		)
+	)
+	(wire
+		(pts
 			(xy 127 135.89) (xy 129.54 135.89)
 		)
@@
 		)
 	)
+	(global_label "VDDSW"
+		(shape bidirectional)
+		(at 69.85 22.86 180)
+		(fields_autoplaced yes)
+		(effects
+			(font
+				(size 1.27 1.27)
+			)
+			(justify right)
+		)
+		(property "Intersheetrefs" "${INTERSHEET_REFS}"
+			(at 59.464 22.86 0)
+			(effects
+				(font
+					(size 1.27 1.27)
+				)
+				(justify right)
+				(hide yes)
+			)
+		)
+	)
 	(global_label "TMS"
 		(shape output)
@@
 			)
 		)
-		(property "Footprint" ""
+		(property "Footprint" "Resistor_SMD:R_0402_1005Metric"
 			(at 133.35 137.668 90)
 			(effects
@@
 			)
 		)
-		(property "Footprint" ""
+		(property "Footprint" "Library:D0430G02V01"
 			(at 158.496 137.414 0)
 			(effects
@@
 			)
 		)
-		(property "Footprint" ""
+		(property "Footprint" "Capacitor_SMD:C_0402_1005Metric"
 			(at 122.8852 110.49 0)
 			(effects
@@
 			)
 		)
-		(property "Footprint" ""
+		(property "Footprint" "Connector:Tag-Connect_TC2050-IDC-NL_2x05_P1.27mm_Vertical_with_bottom_clip"
 			(at 44.45 76.2 0)
 			(effects
@@
 			)
 		)
-		(property "Footprint" ""
+		(property "Footprint" "Resistor_SMD:R_0402_1005Metric"
 			(at 89.662 49.53 90)
 			(effects
@@
 			)
 		)
-		(property "Footprint" ""
+		(property "Footprint" "Resistor_SMD:R_0402_1005Metric"
 			(at 82.042 49.53 90)
 			(effects
@@
 			)
 		)
-		(property "Footprint" ""
+		(property "Footprint" "Capacitor_SMD:C_0402_1005Metric"
 			(at 115.2652 110.49 0)
 			(effects

Commit message: Work on pcb layout, added no fill zones
Parts:
- removed J1: U.FL, Connector_Coaxial:U.FL_Molex_MCRF_73412-0110_Vertical, symbol Connector:Conn_Coaxial
- removed R1: 680, Resistor_SMD:R_0402_1005Metric, symbol Device:R
- added R1: 0, Resistor_SMD:R_0402_1005Metric, symbol Device:R_Small
- U1: footprint Package_DFN_QFN:Texas_RTW_WQFN-24-1EP_4x4mm_P0.5mm_EP2.7x2.7mm_ThermalVias -> tcal:WQFN24_RTW-J_TEX-L
Connections:
- net at U1.8 (P07): now also R1.1
- net at U2.1 (COM): now also R1.2
Other:
- note added: "Pad for current limiting resistor"
Changed lines of the file:
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@@
 	)
 	(junction
-		(at 251.46 41.91)
-		(diameter 0)
-		(color 0 0 0 0)
-	)
-	(junction
 		(at 114.3 101.6)
 		(diameter 0)
@@
 	)
 	(junction
-		(at 256.54 49.53)
-		(diameter 0)
-		(color 0 0 0 0)
-	)
-	(junction
 		(at 83.82 60.96)
 		(diameter 0)
@@
 	(wire
 		(pts
-			(xy 127 135.89) (xy 129.54 135.89)
+			(xy 127 135.89) (xy 130.81 135.89)
 		)
 		(stroke
@@
 	(wire
 		(pts
+			(xy 135.89 135.89) (xy 139.7 135.89)
+		)
+		(stroke
+			(width 0)
+			(type default)
+		)
+	)
+	(wire
+		(pts
 			(xy 127 143.51) (xy 139.7 143.51)
 		)
@@
 	(wire
 		(pts
-			(xy 251.46 41.91) (xy 251.46 44.45)
-		)
-		(stroke
-			(width 0)
-			(type default)
-		)
-	)
-	(wire
-		(pts
 			(xy 88.9 156.21) (xy 88.9 158.75)
 		)
@@
 	(wire
 		(pts
-			(xy 264.16 49.53) (xy 256.54 49.53)
+			(xy 248.92 49.53) (xy 264.16 49.53)
 		)
 		(stroke
@@
 	(wire
 		(pts
-			(xy 137.16 135.89) (xy 139.7 135.89)
-		)
-		(stroke
-			(width 0)
-			(type default)
-		)
-	)
-	(wire
-		(pts
-			(xy 264.16 41.91) (xy 251.46 41.91)
-		)
-		(stroke
-			(width 0)
-			(type default)
-		)
-	)
-	(wire
-		(pts
-			(xy 248.92 49.53) (xy 256.54 49.53)
-		)
-		(stroke
-			(width 0)
-			(type default)
-		)
-	)
-	(wire
-		(pts
 			(xy 127 120.65) (xy 139.7 120.65)
 		)
@@
 	(wire
 		(pts
-			(xy 251.46 41.91) (xy 248.92 41.91)
+			(xy 248.92 41.91) (xy 264.16 41.91)
 		)
 		(stroke
@@
 		)
 	)
+	(text "Pad for current limiting\nresistor"
+		(exclude_from_sim no)
+		(at 133.35 138.684 0)
+		(effects
+			(font
+				(size 1.27 1.27)
+			)
+		)
+	)
 	(text "I2c pull-up resisstors"
 		(exclude_from_sim no)
@@
 		)
 		(property "Value" "DNP"
-			(at 236.22 49.53 90)
+			(at 236.474 49.276 90)
 			(effects
 				(font
@@
 	)
 	(symbol
-		(lib_id "Device:R")
-		(at 133.35 135.89 90)
-		(unit 1)
-		(exclude_from_sim no)
-		(in_bom yes)
-		(on_board yes)
-		(dnp no)
-		(property "Reference" "R1"
-			(at 131.318 138.684 90)
-			(effects
-				(font
-					(size 1.27 1.27)
-				)
-			)
-		)
-		(property "Value" "680"
-			(at 135.382 138.684 90)
-			(effects
-				(font
-					(size 1.27 1.27)
-				)
-			)
-		)
-		(property "Footprint" "Resistor_SMD:R_0402_1005Metric"
-			(at 133.35 137.668 90)
-			(effects
-				(font
-					(size 1.27 1.27)
-				)
-				(hide yes)
-			)
-		)
-		(property "Datasheet" "~"
-			(at 133.35 135.89 0)
-			(effects
-				(font
-					(size 1.27 1.27)
-				)
-				(hide yes)
-			)
-		)
-		(property "Description" "Resistor"
-			(at 133.35 135.89 0)
-			(effects
-				(font
-					(size 1.27 1.27)
-				)
-				(hide yes)
-			)
-		)
-		(pin "2"
-		)
-		(pin "1"
-		)
-		(instances
-			(project ""
-				(path "/e96f5edd-89b2-41c9-95e7-7ba29a607891"
-					(reference "R1")
-					(unit 1)
-				)
-			)
-		)
-	)
-	(symbol
 		(lib_id "power:GND")
 		(at 113.03 27.94 270)
@@
 		)
 		(property "Value" "DNP"
-			(at 236.22 52.07 90)
+			(at 236.474 52.07 90)
 			(effects
 				(font
@@
 			)
 		)
-		(property "Footprint" "Package_DFN_QFN:Texas_RTW_WQFN-24-1EP_4x4mm_P0.5mm_EP2.7x2.7mm_ThermalVias"
+		(property "Footprint" "tcal:WQFN24_RTW-J_TEX-L"
 			(at 117.348 164.592 0)
 			(effects
@@
 	)
 	(symbol
+		(lib_id "Device:R_Small")
+		(at 133.35 135.89 90)
+		(unit 1)
+		(exclude_from_sim no)
+		(in_bom yes)
+		(on_board yes)
+		(dnp no)
+		(property "Reference" "R1"
+			(at 129.54 134.366 90)
+			(effects
+				(font
+					(size 1.27 1.27)
+				)
+			)
+		)
+		(property "Value" "0"
+			(at 136.144 134.62 90)
+			(effects
+				(font
+					(size 1.27 1.27)
+				)
+			)
+		)
+		(property "Footprint" "Resistor_SMD:R_0402_1005Metric"
+			(at 133.35 135.89 0)
+			(effects
+				(font
+					(size 1.27 1.27)
+				)
+				(hide yes)
+			)
+		)
+		(property "Datasheet" "~"
+			(at 133.35 135.89 0)
+			(effects
+				(font
+					(size 1.27 1.27)
+				)
+				(hide yes)
+			)
+		)
+		(property "Description" "Resistor, small symbol"
+			(at 133.35 135.89 0)
+			(effects
+				(font
+					(size 1.27 1.27)
+				)
+				(hide yes)
+			)
+		)
+		(pin "2"
+		)
+		(pin "1"
+		)
+		(instances
+			(project ""
+				(path "/e96f5edd-89b2-41c9-95e7-7ba29a607891"
+					(reference "R1")
+					(unit 1)
+				)
+			)
+		)
+	)
+	(symbol
 		(lib_id "Tag-Connect:TC2050-IDC-430")
 		(at 44.45 76.2 0)
@@
 					(unit 1)
 				)
-			)
-		)
-	)
-	(symbol
-		(lib_id "Connector:Conn_Coaxial")
-		(at 256.54 44.45 0)
-		(unit 1)
-		(exclude_from_sim no)
-		(in_bom yes)
-		(on_board yes)
-		(dnp no)
-		(property "Reference" "J1"
-			(at 256.54 48.26 0)
-			(effects
-				(font
-					(size 1.27 1.27)
-				)
-				(justify left)
-			)
-		)
-		(property "Value" "U.FL"
-			(at 251.46 46.99 0)
-			(effects
-				(font
-					(size 1.27 1.27)
-				)
-				(justify left)
-			)
-		)
-		(property "Footprint" "Connector_Coaxial:U.FL_Molex_MCRF_73412-0110_Vertical"
-			(at 256.54 44.45 0)
-			(effects
-				(font
-					(size 1.27 1.27)
-				)
-				(hide yes)
-			)
-		)
-		(property "Datasheet" "~"
-			(at 256.54 44.45 0)
-			(effects
-				(font
-					(size 1.27 1.27)
-				)
-				(hide yes)
-			)
-		)
-		(property "Description" ""
-			(at 256.54 44.45 0)
-			(effects
-				(font
-					(size 1.27 1.27)
-				)
-				(hide yes)
-			)
-		)
-		(pin "1"
-		)
-		(pin "2"
-		)
-		(instances
-			(project "tcg_counter"
-				(path "/e96f5edd-89b2-41c9-95e7-7ba29a607891"
-					(reference "J1")
-					(unit 1)
-				)

Commit message: Added tagconnect power signals
Connections:
- net VDDSW: now also P1.2 (VCC_Tool)
- net VDDB: now reaches C1.1, U3.4 (VDDB)
- net VDDB: now also P1.6 (NC)
Other:
- note added: "TagConnect JTAG signals are 1.5V levels converted on offboard translator board. VDDB is connected to VDDSW only when the tagconnect cable is plugged in."
Changed lines of the file:
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@@
+	)
+	(junction
+		(at 125.73 38.1)
+		(diameter 0)
+		(color 0 0 0 0)
 	)
 	(junction
@@
 	(wire
 		(pts
+			(xy 125.73 35.56) (xy 125.73 38.1)
+		)
+		(stroke
+			(width 0)
+			(type default)
+		)
+	)
+	(wire
+		(pts
 			(xy 127 33.02) (xy 120.65 33.02)
 		)
@@
 	(wire
 		(pts
+			(xy 55.88 81.28) (xy 60.96 81.28)
+		)
+		(stroke
+			(width 0)
+			(type default)
+		)
+	)
+	(wire
+		(pts
 			(xy 69.85 22.86) (xy 74.93 22.86)
 		)
@@
 	(wire
 		(pts
+			(xy 125.73 38.1) (xy 127 38.1)
+		)
+		(stroke
+			(width 0)
+			(type default)
+		)
+	)
+	(wire
+		(pts
 			(xy 242.57 76.2) (xy 240.03 76.2)
 		)
@@
 	(wire
 		(pts
-			(xy 120.65 38.1) (xy 127 38.1)
+			(xy 120.65 38.1) (xy 125.73 38.1)
 		)
 		(stroke
@@
 	(wire
 		(pts
+			(xy 104.14 35.56) (xy 125.73 35.56)
+		)
+		(stroke
+			(width 0)
+			(type default)
+		)
+	)
+	(wire
+		(pts
 			(xy 127 153.67) (xy 139.7 153.67)
 		)
@@
 		(pts
 			(xy 109.22 168.91) (xy 109.22 172.72)
+		)
+		(stroke
+			(width 0)
+			(type default)
+		)
+	)
+	(wire
+		(pts
+			(xy 25.4 73.66) (xy 33.02 73.66)
 		)
 		(stroke
@@
 		(exclude_from_sim no)
 		(at 88.392 44.45 0)
+		(effects
+			(font
+				(size 1.27 1.27)
+			)
+		)
+	)
+	(text "TagConnect JTAG signals are 1.5V levels converted on offboard translator board. \nVDDB is connected to VDDSW only when the tagconnect cable is plugged in."
+		(exclude_from_sim no)
+		(at 40.894 56.388 0)
 		(effects
 			(font
@@
 		)
 	)
+	(global_label "VDDB"
+		(shape bidirectional)
+		(at 60.96 81.28 0)
+		(fields_autoplaced yes)
+		(effects
+			(font
+				(size 1.27 1.27)
+			)
+			(justify left)
+		)
+		(property "Intersheetrefs" "${INTERSHEET_REFS}"
+			(at 69.9551 81.28 0)
+			(effects
+				(font
+					(size 1.27 1.27)
+				)
+				(justify left)
+				(hide yes)
+			)
+		)
+	)
 	(global_label "TDI"
 		(shape input)
@@
 			(effects
 				(font
+					(size 1.27 1.27)
+				)
+				(justify right)
+				(hide yes)
+			)
+		)
+	)
+	(global_label "VDDB"
+		(shape bidirectional)
+		(at 104.14 35.56 180)
+		(fields_autoplaced yes)
+		(effects
+			(font
+				(size 1.27 1.27)
+			)
+			(justify right)
+		)
+		(property "Intersheetrefs" "${INTERSHEET_REFS}"
+			(at 95.1449 35.56 0)
+			(effects
+				(font
+					(size 1.27 1.27)
+				)
+				(justify right)
+				(hide yes)
+			)
+		)
+	)
+	(global_label "VDDSW"
+		(shape output)
+		(at 25.4 73.66 180)
+		(fields_autoplaced yes)
+		(effects
+			(font
+				(size 1.27 1.27)
+			)
+			(justify right)
+		)
+		(property "Intersheetrefs" "${INTERSHEET_REFS}"
+			(at 16.1253 73.66 0)
+			(effects
+				(font
