File: tcg_counter/tcg_counter.kicad_sch (KiCad schematic)
At the start: 20 parts, among them P1 TC2050-IDC-430, U1 TCAL9539RTW, U3 RF430FRL152

Commit message: v1.0 hardware revision
Parts:
- U1: footprint tcal:WQFN24_RTW-J_TEX-L -> TIFootprints:TI_RTW24_4x4mm_EP2.2mm
- renumbered U2 to DS1, R4 to R2, R5 to R3, U3 to U2
Changed lines of the file:
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@@
 		(on_board yes)
 		(dnp no)
-		(property "Reference" "U2"
+		(property "Reference" "DS1"
 			(at 157.48 113.03 0)
 			(effects
@@
 			(project ""
 				(path "/e96f5edd-89b2-41c9-95e7-7ba29a607891"
-					(reference "U2")
+					(reference "DS1")
 					(unit 1)
 				)
@@
 		(on_board yes)
 		(dnp no)
-		(property "Reference" "U3"
+		(property "Reference" "U2"
 			(at 177.8 18.1356 0)
 			(effects
@@
 			(project "tcg_counter"
 				(path "/e96f5edd-89b2-41c9-95e7-7ba29a607891"
-					(reference "U3")
+					(reference "U2")
 					(unit 1)
 				)
@@
 			)
 		)
-		(property "Footprint" "tcal:WQFN24_RTW-J_TEX-L"
+		(property "Footprint" "TIFootprints:TI_RTW24_4x4mm_EP2.2mm"
 			(at 117.348 164.592 0)
 			(effects
@@
 		(on_board yes)
 		(dnp no)
-		(property "Reference" "R4"
+		(property "Reference" "R2"
 			(at 93.218 48.26 0)
 			(effects
@@
 			(project ""
 				(path "/e96f5edd-89b2-41c9-95e7-7ba29a607891"
-					(reference "R4")
+					(reference "R2")
 					(unit 1)
 				)
@@
 		(on_board yes)
 		(dnp no)
-		(property "Reference" "R5"
+		(property "Reference" "R3"
 			(at 85.344 48.26 0)
 			(effects
@@
 			(project ""
 				(path "/e96f5edd-89b2-41c9-95e7-7ba29a607891"
-					(reference "R5")
-					(unit 1)
-				)
+					(reference "R3")
+					(unit 1)
+				)
