File: tcg_counter/_autosave-tcg_counter.kicad_sch (KiCad schematic)
At the start: 20 parts, among them P1 TC2050-IDC-430, U1 TCAL9539RTW, U3 RF430FRL152

Commit message: Finished traces, made new footprint for TCAL9539
Parts:
- U1: footprint tcal:WQFN24_RTW-J_TEX-L -> TIFootprints:TI_RTW24_4x4mm_EP2.2mm
Changed lines of the file:
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@@
 			)
 		)
-		(property "Footprint" "tcal:WQFN24_RTW-J_TEX-L"
+		(property "Footprint" "TIFootprints:TI_RTW24_4x4mm_EP2.2mm"
 			(at 117.348 164.592 0)
 			(effects
